File: Particle-Gateway.brd (EAGLE design)
At the start: 47 x 40.6 mm, 25 parts, among them J2 GROVE-I2C, J3 Lipo Battery, J4 GROVE-I2C, J5 CON_HEADER_1X08-PTH, P1 PADSMALL, U1 AMS1117-3.3

Commit message: Adjusted SMA connector exposed PAD
Parts:
- added J$1: SMA_EDGE, SparkFun-Connectors:SMA-EDGE
- added U$1: (no value), _c2h:LOGO_CH2I_75MM
- moved U-FL 6.47 mm to (9.05, 2.00), turned to 90 degrees
- moved R19 2.62 mm to (14.6, 3.43), turned to 270 degrees
- moved P1 2.22 mm to (7.59, 6.06)
- moved R20 0.81 mm to (17.1, 3.43), turned to 270 degrees
Connections:
- net ANT: now also J$1.SIG
- net GND: now also J$1.GND@0, J$1.GND@1, J$1.GND@2, J$1.GND@3
Routing:
- net SCL: track 91.0 -> 84.7 mm
- net ANT: track 16.0 -> 21.7 mm
- net GND: track 6.87 -> 2.74 mm, vias 9 -> 10
- net SDA: track 82.4 -> 79.2 mm
- net 3V3-REG: track 147.2 -> 145.0 mm, vias 3 -> 2
- net N$5: track 2.07 -> 0.00 mm
Other:
- board text added: "Particle Gateway http://hallard.me"
- board text added: "V1.0a"
- board text removed: "RF Ant"
- board text removed: "Spark Gateway V1.0 http://hallard.me"
